Commit message: Let the rover turn, and stop the lidar scanning its own mast
Two defects that both fed the SLAM map instability.

1. The rover could not rotate at all. A pure yaw command counter-rotated
   the wheels correctly (-1.71 / +1.71 rad/s) and the rover turned 0
   degrees against the ~143 commanded. Cause was the previous friction
   commit: it set mu2 to 2.0 along with mu, and mu2 is the LATERAL
   coefficient. A six-wheel skid steer turns by scrubbing its wheels
   sideways, so high mu2 welds it to a straight line. mu stays 1.5 for
   traction, mu2 drops to 0.1. The rover now turns 122.8 degrees (the
   shortfall is ordinary scrub loss) and still drives 1.46 m forward.

   This also corrupted SLAM on its own: odometry reported rotation that
   never physically happened, so the scan matcher was fighting its own
   odometry prior.

2. The lidar was buried inside the camera mast. lidar_monitor reported
   front = 0.13 m constantly -- the mast sat at the same x as the lidar
   and spanned z 0.09-0.35, straddling the scan plane at z=0.11, so a
   large part of every scan was a fixed return off the rover itself. A
   scan matcher cannot localise against geometry that never moves
   relative to the sensor. The lidar moves up to z=0.42, clear of
   everything on the rover; the mast moves back and down. Forward range
   went from 0.13 m to over 1 m.

   The wheel roll also moves from the link pose onto the geometry here,
   for the same reason as the preceding edubot commit.

SDF and URDF are kept in step, so RViz still draws what Gazebo simulates.

NOT FIXED by this commit: the reported symptom of the SLAM map rotating
around the rover still reproduces after both changes -- map->odom still
swings tens of degrees across a few curves. These are two genuine defects
removed from the path, not the root cause. Next step is to run the same
rover with SLAM in the classroom: if the map is stable there and spins on
Mars, the terrain lacks the stable vertical structure scan matching needs
and the fix belongs in the world, not the robot.

Co-Authored-By: Claude Opus 5 (1M context) <noreply@anthropic.com>

File: src/edu_bringup/models/rover.urdf.xacro (robot description, xacro)
@@ -103,5 +103,5 @@
     <parent link="base_link"/>
     <child  link="mast_link"/>
-    <origin xyz="0.15 0 0.22" rpy="0 0 0"/>
+    <origin xyz="-0.12 0 0.18" rpy="0 0 0"/>
   </joint>
   <!-- Sensor frames. Positions match model.sdf. -->
@@ -119,5 +119,5 @@
     <parent link="base_link"/>
     <child  link="lidar_link"/>
-    <origin xyz="0.15 0 0.11" rpy="0 0 0"/>
+    <origin xyz="0.15 0 0.42" rpy="0 0 0"/>
   </joint>
   <link name="camera_link">
@@ -134,5 +134,5 @@
     <parent link="base_link"/>
     <child  link="camera_link"/>
-    <origin xyz="0.17 0 0.37" rpy="0 0 0"/>
+    <origin xyz="-0.10 0 0.33" rpy="0 0 0"/>
   </joint>
   <link name="imu_link">

Commit message: Add a 3-D lidar so RViz can show terrain, not just the flat map
The SLAM map is a 2-D occupancy grid: free/occupied, no height. Asking it
to show the craters and ridge is asking for something it does not
contain, and the single horizontal lidar at z=0.42 cannot supply it
either -- one plane sees one slice.

The rover now carries a SECOND lidar with 16 vertical rays over +/- 15
degrees, tilted down, publishing a PointCloud2 on /points/points at 5 Hz.
Displayed in RViz with AxisColor on Z it draws the terrain coloured by
height, beside the flat map rather than instead of it.

Deliberately a separate sensor: slam_toolbox wants a single-plane
LaserScan, and adding vertical rays to /scan would break the map. /scan
is untouched, so mapping behaves exactly as before.

The topic name is the part worth knowing. A gpu_lidar publishes TWO
topics -- <topic> as a LaserScan and <topic>/points as the cloud -- so a
sensor whose <topic> is 'points' puts its cloud on /points/points.
Bridging /points as PointCloudPacked is a type mismatch against the
LaserScan that actually lives there, and it fails the way QoS mismatches
do: the ROS topic appears in `ros2 topic list` and never carries a
message, with no error anywhere. That cost a debugging round here and is
commented at the bridge line so it does not cost another.

16 x 180 points at 5 Hz is sized for software rendering; raising either
number is the first thing that will cost frame rate.

Co-Authored-By: Claude Opus 5 (1M context) <noreply@anthropic.com>

File: src/edu_bringup/models/rover.urdf.xacro (robot description, xacro)
@@ -116,4 +116,21 @@
     </inertial>
   </link>
+  <!-- 3-D lidar used for terrain visualisation (publishes /points).
+       Pose and tilt must match model.sdf. -->
+  <link name="lidar3d_link">
+    <visual>
+      <geometry><cylinder radius="0.03" length="0.03"/></geometry>
+      <material name="blue3d"><color rgba="0.2 0.4 0.9 1"/></material>
+    </visual>
+    <inertial>
+      <mass value="0.1"/>
+      <inertia ixx="4e-5" ixy="0" ixz="0" iyy="4e-5" iyz="0" izz="4e-5"/>
+    </inertial>
+  </link>
+  <joint name="lidar3d_joint" type="fixed">
+    <parent link="base_link"/>
+    <child  link="lidar3d_link"/>
+    <origin xyz="0.15 0 0.38" rpy="0 0.15 0"/>
+  </joint>
   <joint name="lidar_joint" type="fixed">
     <parent link="base_link"/>

Commit message: Fix the rover camera and flicker; add no-go hills and sharper craters
Three things, from the screenshots.

THE CAMERA WAS LOOKING AT ITS OWN MAST. The rover-cam view was mostly a
blue cylinder with a red block above it. When the mast moved back to
x=-0.12 to clear the lidar, the camera stayed at x=-0.10 -- 2 cm from the
mast centre, i.e. inside it. It moves to x=-0.04, z=0.40, in front of the
mast and above the deck, tilted 0.1 rad down so it frames the terrain
rather than the horizon. Same bug as the lidar one, missed because I
fixed the sensor I was looking at and did not check the other.

THE FLICKER was the deck plate: a 0.02 m slab at z=0.08 left its
underside 1 cm above the 0.06 chassis top. Under software rendering the
depth buffer could not separate them, so the surfaces fought every frame
-- and being geometry, it showed in Gazebo, the camera and RViz alike,
which is what made it look like three separate faults. The deck drops to
z=0.075.

TERRAIN. make_heightmap.py gains a mound() for steep hills -- gaussian
rather than cosine falloff, so the flanks keep rising and the rover loses
traction partway up instead of cresting them. Five of those as no-go
areas, plus five small sharp craters (tight radius, large depth) that
read as pits to drive around rather than dishes to roll through, and a
crater pair whose shared rim makes a natural narrow pass. Mounds are
applied before craters so a crater on a slope still digs in.

Regenerating the terrain invalidates every rock's hand-set z: three had
drifted more than half a metre and would have been visibly floating.
reseat_rocks.py recomputes them from heightmap.png and rewrites the poses
in place, so this is repeatable rather than 40 numbers to re-derive by
hand. It reuses make_terrain_mesh.py's exact mapping including the row
inversion (image row 0 is +y) -- without that the lookup is mirrored
north/south and every rock sits at the height of the wrong side of the
map, which is wrong in a way that still looks plausible.

Co-Authored-By: Claude Opus 5 (1M context) <noreply@anthropic.com>

File: src/edu_bringup/models/rover.urdf.xacro (robot description, xacro)
@@ -151,5 +151,5 @@
     <parent link="base_link"/>
     <child  link="camera_link"/>
-    <origin xyz="-0.10 0 0.33" rpy="0 0 0"/>
+    <origin xyz="-0.04 0 0.40" rpy="0 0.10 0"/>
   </joint>
   <link name="imu_link">

Commit message: Make the terrain actually read as terrain, and get the rover out of shot
Two things from the screenshots: the ground looked flat despite having
craters and hills in it, and the camera was still filled by rover
hardware.

TERRAIN WAS TOO GENTLE. The relief was real but tiny -- measured off the
generated mesh, 3.0 m across a 40 m span, a 7.5% grade. Geometrically
present, visually flat. VRANGE 4 -> 12 and SPAN 40 -> 30 gives 9.0 m over
30 m: the mounds are now genuinely unclimbable and the crater notches
visible as notches, which is the point of having put them there.

THE CAMERA WAS LOOKING AT THE LIDARS, not the mast as I assumed when I
moved it last time. Measuring the poses instead of reasoning about them:
the camera sat at x=-0.04 looking along +x, directly into the 2-D lidar
(red, x=0.15 z=0.42) and the 3-D lidar (blue, x=0.15 z=0.38) -- the red
cylinder over a blue one that filled the frame. It moves to x=0.32, past
the deck edge at 0.30, so nothing on the rover is in front of it.

Raising the relief put the ground at the spawn point 2.5 m below zero,
so the hard-coded -z 0.15 would have dropped the rover from a height on
every start. Spawn height now comes from the heightmap, via two
world-conditional spawn nodes: `world` is a LaunchConfiguration and
cannot be branched on in Python, and the classroom's flat plane still
needs the original fixed clearance -- computing a terrain height there
would have buried the EduBot 2.18 m underground.

Verified with --print-description: classroom spawns at 0.15, moon/mars at
-2.18, which matches the measured surface height at (-4,-4).

Co-Authored-By: Claude Opus 5 (1M context) <noreply@anthropic.com>

File: src/edu_bringup/models/rover.urdf.xacro (robot description, xacro)
@@ -151,5 +151,5 @@
     <parent link="base_link"/>
     <child  link="camera_link"/>
-    <origin xyz="-0.04 0 0.40" rpy="0 0.10 0"/>
+    <origin xyz="0.32 0 0.22" rpy="0 0.12 0"/>
   </joint>
   <link name="imu_link">
